File: Eagle Files/RAMPSSB.sch (EAGLE design)
At the start: 30 parts, among them J10 1X2-3.5MM, J7 OSTTH020160, J9 1X2-3.5MM

Commit message: Update for publish
Final update before publish! Get ready!

Still needs some firmware work, but the hardware is there.
Parts:
- removed U$10: M05X2, RepRapjr:M05X2
- added J17, J18, J19: (no value), SparkFun-Retired:CONN_02
- added LED1, LED2: (no value), adafruit:LED3MM
- added R1: (no value), adafruit:R-US_0207/7
- J9: value 1X2-3.5MM -> OSTTH020160; device adafruit:1X2-3.5MM -> con-ost:OSTTH020160
Connections:
- new net LEDGND: LED1.C, LED2.C, R1.1
- new net RX: A-OUT.4, J19.2
- new net TX: A-OUT.3, J19.1
- new net VMOT: J17.1, J18.1, U$6.VMOT, U$7.VMOT
- net +5V: no longer U$10.1
- net GND: now also A-OUT.2, J17.2, J18.2, J9-2.SK, R1.2, SERIAL.2; no longer J9.1
- net VCC: now also J9-1.SK; no longer J9.2
- net XPWM: now also LED1.A
- net YPWM: now also LED2.A
Other:
- note added: "Developed by SZiv"
- note removed: "(C) Scott Ziv"
- moved on the sheet: A-OUT, SERIAL
